Commit message: bien 5

File: src/atom/urdf/atom.xacro (robot description, xacro)
@@ -177,5 +177,5 @@
 	<!-- Color of bot -->
 	<gazebo reference="left_wheel_front">
-		<material>Gazebo/Green</material>
+		<material>Gazebo/Black</material>
 		<kp>1000000.0</kp> <!-- kp and kd for rubber -->
 		<kd>100.0</kd>
@@ -186,5 +186,5 @@
 	</gazebo>
 	<gazebo reference="left_wheel_back">
-		<material>Gazebo/Green</material>
+		<material>Gazebo/Black</material>
 		<kp>1000000.0</kp> <!-- kp and kd for rubber -->
 		<kd>100.0</kd>
@@ -195,5 +195,5 @@
 	</gazebo>
 	<gazebo reference="right_wheel_front">
-		<material>Gazebo/Green</material>
+		<material>Gazebo/Black</material>
 		<kp>1000000.0</kp> <!-- kp and kd for rubber -->
 		<kd>100.0</kd>
@@ -204,34 +204,30 @@
 	</gazebo>
 	<gazebo reference="right_wheel_back">
-		<material>Gazebo/Green</material>
-		<kp>1000000.0</kp> <!-- kp and kd for rubber -->
-		<kd>100.0</kd>
-		<mu1>1.0</mu1>
-		<mu2>1.0</mu2>
-		<maxVel>1.0</maxVel>
-		<minDepth>0.00</minDepth>
-	</gazebo>
-	<!--<gazebo reference="right_wheel">
-		<material>Gazebo/Green</material>
-	</gazebo>-->
+		<material>Gazebo/Black</material>
+		<kp>1000000.0</kp> <!-- kp and kd for rubber -->
+		<kd>100.0</kd>
+		<mu1>1.0</mu1>
+		<mu2>1.0</mu2>
+		<maxVel>1.0</maxVel>
+		<minDepth>0.00</minDepth>
+	</gazebo>
 	<gazebo reference="chassis">
-                        <!-- CAMBIOS AGERGADOS -->
-                <material>Gazebo/Blue</material>
+		<material>Gazebo/Red</material>
 	</gazebo>
   <gazebo>
-    <plugin name="skid_steer_drive_controller" filename="libgazebo_ros_skid_steer_drive.so">
-      <updateRate>10.0</updateRate>
-      <robotNamespace>/1</robotNamespace>
-      <leftFrontJoint>left_wheel_hinge_front</leftFrontJoint>
-      <rightFrontJoint>right_wheel_hinge_front</rightFrontJoint>
-      <leftRearJoint>left_wheel_hinge_back</leftRearJoint>
-      <rightRearJoint>right_wheel_hinge_back</rightRearJoint>
-      <wheelSeparation>0.4</wheelSeparation>
-      <wheelDiameter>0.2</wheelDiameter>
-      <robotBaseFrame>robot_footprint</robotBaseFrame>
-      <torque>10</torque>
-      <topicName>cmd_vel</topicName>
-      <broadcastTF>False</broadcastTF>
-    </plugin>
+	    <plugin name="skid_steer_drive_controller" filename="libgazebo_ros_skid_steer_drive.so">
+	      <updateRate>10.0</updateRate>
+	      <robotNamespace>/</robotNamespace>
+	      <leftFrontJoint>left_wheel_hinge_front</leftFrontJoint>
+	      <rightFrontJoint>right_wheel_hinge_front</rightFrontJoint>
+	      <leftRearJoint>left_wheel_hinge_back</leftRearJoint>
+	      <rightRearJoint>right_wheel_hinge_back</rightRearJoint>
+	      <wheelSeparation>0.4</wheelSeparation>
+	      <wheelDiameter>0.2</wheelDiameter>
+	      <robotBaseFrame>robot_footprint</robotBaseFrame>
+	      <torque>10</torque>
+	      <topicName>cmd_vel</topicName>
+	      <broadcastTF>False</broadcastTF>
+	    </plugin>
   </gazebo>
 </robot>

Commit message: el param de description tiene que ir en robots.launch o no fuciona

File: src/atom/urdf/atom.xacro (robot description, xacro)
@@ -213,10 +213,10 @@
 	</gazebo>
 	<gazebo reference="chassis">
-		<material>Gazebo/Red</material>
+		<material>Gazebo/Green</material>
 	</gazebo>
   <gazebo>
 	    <plugin name="skid_steer_drive_controller" filename="libgazebo_ros_skid_steer_drive.so">
 	      <updateRate>10.0</updateRate>
-	      <robotNamespace>/1</robotNamespace>
+	      <robotNamespace>/</robotNamespace>
 	      <leftFrontJoint>left_wheel_hinge_front</leftFrontJoint>
 	      <rightFrontJoint>right_wheel_hinge_front</rightFrontJoint>

Commit message: Se agrega codigo para controlar robot individualmente, y estan bien separados

File: src/atom/urdf/atom.xacro (robot description, xacro)
@@ -213,10 +213,18 @@
 	</gazebo>
 	<gazebo reference="chassis">
-		<material>Gazebo/Green</material>
+		<material>Gazebo/Red</material>
+		<!--
+  	<material>
+            <script>
+              <uri>/home/jazmin/MultiRobots/src/atom/materials/scripts</uri>
+              <uri>/home/jazmin/MultiRobots/src/atom/materials/textures</uri>
+              <name>R1/Diffuse</name>
+            </script>
+          </material>
+          -->
 	</gazebo>
   <gazebo>
 	    <plugin name="skid_steer_drive_controller" filename="libgazebo_ros_skid_steer_drive.so">
 	      <updateRate>10.0</updateRate>
-	      <robotNamespace>/</robotNamespace>
 	      <leftFrontJoint>left_wheel_hinge_front</leftFrontJoint>
 	      <rightFrontJoint>right_wheel_hinge_front</rightFrontJoint>

Commit message: obtengo la info de poses y velocidades y pasan a csv, archivo MoverRobots sirve para cambiar la vel, puedo unirlos

File: src/atom/urdf/atom.xacro (robot description, xacro)
@@ -10,4 +10,5 @@
 	<xacro:property name="robot_wheel_length" value="0.05"/>
 	<xacro:property name="robot_wheel_radius" value="0.1"/>
+	<xacro:property name="hokoyu_mass" value="1e-5"/>
 	<!-- Make Chassis of Bot -->
 	<link name="chassis">
@@ -131,4 +132,28 @@
 		</collision>
 	</link>
+	<!-- Hokuyo Lidar -->
+	<link name="hokuyo">
+		<inertial>
+			<mass value="${hokoyu_mass}"/>
+			<origin xyz="0 0 0" rpy="0 0 0"/>
+			<inertia
+		        ixx="1e-6" ixy="0.0" ixz="0.0"
+		        iyy="1e-6" iyz="0.0"
+		        izz="1e-6"
+		      />
+		</inertial>
+		<visual>
+			<origin xyz="0 0 0" rpy="0 0 0"/>
+			<geometry>
+				<mesh filename="/home/jazmin/MultiRobots/src/atom/urdf/hokuyo.dae"/>
+			</geometry>
+		</visual>
+		<collision>
+			<origin xyz="0 0 0" rpy="0 0 0"/>
+			<geometry>
+				<box size="0.1 0.1 0.1"/>
+			</geometry>
+		</collision>
+	</link>
 	<!-- Project center to the ground -->
 	<link name="robot_footprint"></link>
@@ -174,4 +199,11 @@
 		<parent link="robot_footprint"/>
 		<child link="chassis" />
+	</joint>
+	<!-- Hokoyu Joint -->
+	<joint name="hokuyo_joint" type="fixed">
+	    <origin xyz="0.2 0 0.2" rpy="0 0 0" />
+	    <parent link="chassis"/>
+	    <child link="hokuyo" />
+	    <axis xyz="0 1 0"/>
 	</joint>
 	<!-- Color of bot -->
@@ -224,18 +256,5 @@
           -->
 	</gazebo>
-  <gazebo>
-	    <plugin name="skid_steer_drive_controller" filename="libgazebo_ros_skid_steer_drive.so">
-	      <updateRate>10.0</updateRate>
-	      <leftFrontJoint>left_wheel_hinge_front</leftFrontJoint>
-	      <rightFrontJoint>right_wheel_hinge_front</rightFrontJoint>
-	      <leftRearJoint>left_wheel_hinge_back</leftRearJoint>
-	      <rightRearJoint>right_wheel_hinge_back</rightRearJoint>
-	      <wheelSeparation>0.4</wheelSeparation>
-	      <wheelDiameter>0.2</wheelDiameter>
-	      <robotBaseFrame>robot_footprint</robotBaseFrame>
-	      <torque>10</torque>
-	      <topicName>cmd_vel</topicName>
-	      <broadcastTF>False</broadcastTF>
-	    </plugin>
-  </gazebo>
+	<!-- Motor, Camera and Lidar Simulation -->
+<xacro:include filename="$(find atom)/urdf/atom.gazebo" />
 </robot>
